Commit message: feat: import where_am_i project and adapt to this one

File: map_my_world/urdf/my_robot.xacro (robot description, xacro)
@@ -1,5 +1,6 @@
 <?xml version='1.0'?>
-<robot name="my_robot" xmlns:xacro="http://www.ros.org/wiki/xacro">
-  <xacro:include filename="$(find where_am_i)/urdf/my_robot.gazebo" />
+<robot name="my_robot"
+  xmlns:xacro="http://www.ros.org/wiki/xacro">
+  <xacro:include filename="$(find map_my_world)/urdf/my_robot.gazebo" />
   <material name="blue">
     <color rgba="0 0 0.8 1"/>
@@ -23,14 +24,10 @@
       <mass value="15.0"/>
       <origin xyz="0.0 0 0" rpy=" 0 0 0"/>
-      <inertia
-          ixx="0.1" ixy="0" ixz="0"
-          iyy="0.1" iyz="0"
-          izz="0.1"
-      />
+      <inertia ixx="0.1" ixy="0" ixz="0" iyy="0.1" iyz="0" izz="0.1" />
     </inertial>
     <collision name='collision'>
       <origin xyz="0 0 0" rpy=" 0 0 0"/>
       <geometry>
-          <cylinder radius="0.15" length="0.1"/>
+        <cylinder radius="0.15" length="0.1"/>
       </geometry>
     </collision>
@@ -69,26 +66,22 @@
   <!-- Left wheel -->
   <link name='left_wheel'>
-      <inertial>
-        <mass value="5.0"/>
-        <origin xyz="0.0 0 0" rpy="0 1.5707 1.5707"/>
-        <inertia
-            ixx="0.1" ixy="0" ixz="0"
-            iyy="0.1" iyz="0"
-            izz="0.1"
-        />
-      </inertial>
-      <collision>
-        <origin xyz="0 0 0" rpy="0 1.5707 1.5707"/>
-        <geometry>
-          <cylinder radius="0.1" length="0.05"/>
-        </geometry>
-      </collision>
-      <visual>
-        <origin xyz="0 0 0" rpy="0 1.5707 1.5707"/>
-        <geometry>
-          <cylinder radius="0.1" length="0.05"/>
-        </geometry>
-        <material name="red"/>
-      </visual>
+    <inertial>
+      <mass value="5.0"/>
+      <origin xyz="0.0 0 0" rpy="0 1.5707 1.5707"/>
+      <inertia ixx="0.1" ixy="0" ixz="0" iyy="0.1" iyz="0" izz="0.1" />
+    </inertial>
+    <collision>
+      <origin xyz="0 0 0" rpy="0 1.5707 1.5707"/>
+      <geometry>
+        <cylinder radius="0.1" length="0.05"/>
+      </geometry>
+    </collision>
+    <visual>
+      <origin xyz="0 0 0" rpy="0 1.5707 1.5707"/>
+      <geometry>
+        <cylinder radius="0.1" length="0.05"/>
+      </geometry>
+      <material name="red"/>
+    </visual>
   </link>
   <joint type="continuous" name="left_wheel_hinge">
@@ -105,9 +98,5 @@
       <mass value="5.0"/>
       <origin xyz="0.0 0 0" rpy="0 1.5707 1.5707"/>
-      <inertia
-          ixx="0.1" ixy="0" ixz="0"
-          iyy="0.1" iyz="0"
-          izz="0.1"
-      />
+      <inertia ixx="0.1" ixy="0" ixz="0" iyy="0.1" iyz="0" izz="0.1" />
     </inertial>
     <collision>
@@ -176,5 +165,5 @@
       <origin xyz="0.0 0 0" rpy="0 0 0"/>
       <geometry>
-        <mesh filename="package://where_am_i/meshes/hokuyo.dae"/>
+        <mesh filename="package://map_my_world/meshes/hokuyo.dae"/>
       </geometry>
     </visual>
@@ -186,3 +175,10 @@
     <axis xyz="0 1 0" rpy="0 0 0"/>
   </joint>
+  <joint name="camera_optical_joint" type="fixed">
+    <origin xyz="0 0 0" rpy="-1.5707 0 -1.5707"/>
+    <parent link="camera"/>
+    <child link="camera_link_optical"/>
+  </joint>
+  <link name="camera_link_optical">
+  </link>
 </robot>

Commit message: docs: rename bare pkg to new one

File: map_my_world/urdf/my_robot.xacro (robot description, xacro)
@@ -2,5 +2,5 @@
 <robot name="my_robot"
   xmlns:xacro="http://www.ros.org/wiki/xacro">
-  <xacro:include filename="$(find map_my_world)/urdf/my_robot.gazebo" />
+  <xacro:include filename="$(find home_service_robot)/urdf/my_robot.gazebo" />
   <material name="blue">
     <color rgba="0 0 0.8 1"/>
@@ -165,5 +165,5 @@
       <origin xyz="0.0 0 0" rpy="0 0 0"/>
       <geometry>
-        <mesh filename="package://map_my_world/meshes/hokuyo.dae"/>
+        <mesh filename="package://home_service_robot/meshes/hokuyo.dae"/>
       </geometry>
     </visual>
